File: Hardware/KiCad/C64 USB-C PD Power Adapter.kicad_sch (KiCad schematic)
At the start: 39 parts, among them J1 USB-C (power in), J2 C64 POWER (DIN-7 male), Q1 AO3401A, U1 CH224A, U2 TPS54302DDCR, U3 TPS54302DDCR

Commit message: v0.3: cut JLC extended parts from 15 to 4, 0603 passives
All 0402 parts moved to 0603 JLC Basic; TVS diodes swapped to Preferred
parts; L1 now the same FXL0530 as L2; PTCs replaced by Basic 0R links
(footprints still take a 1206 PTC); 5 V feedback 75k/10k. Board rebuilt
from the user's placement, re-routed (DRC clean). CPL now carries the
U1-U3 +90 fix confirmed in JLC's preview.

Co-Authored-By: Claude Opus 5.5 <noreply@anthropic.com>
Parts:
- C11, C5: value 100nF -> 100nF/50V; footprint C64_PD_PSU:C_0402_1005Metric -> C64_PD_PSU:C_0603_1608Metric; LCSC C1525 -> C14663
- C14, C8: value 75pF -> 100pF; footprint C64_PD_PSU:C_0402_1005Metric -> C64_PD_PSU:C_0603_1608Metric; LCSC C37809 -> C14858
- D1: LCSC C193402 -> C19077497
- D2: LCSC C353315 -> C41376087
- F1: value 2A -> 0R; footprint C64_PD_PSU:Fuse_1206_3216Metric -> C64_PD_PSU:R_1206_3216Metric; symbol C64_PD_PSU:Polyfuse -> C64_PD_PSU:R; LCSC C22374899 -> C17888
- F2: value 1.1A -> 0R; footprint C64_PD_PSU:Fuse_1206_3216Metric -> C64_PD_PSU:R_1206_3216Metric; symbol C64_PD_PSU:Polyfuse -> C64_PD_PSU:R; LCSC C2798026 -> C17888
- L1: footprint C64_PD_PSU:L_Changjiang_FXL0630 -> C64_PD_PSU:L_Changjiang_FXL0530; LCSC C167223 -> C177248
- R1: footprint C64_PD_PSU:R_0402_1005Metric -> C64_PD_PSU:R_0603_1608Metric; LCSC C25796 -> C23206
- R10, R5: footprint C64_PD_PSU:R_0402_1005Metric -> C64_PD_PSU:R_0603_1608Metric; LCSC C25792 -> C25819
- R11, R2, R3: footprint C64_PD_PSU:R_0402_1005Metric -> C64_PD_PSU:R_0603_1608Metric; LCSC C25741 -> C25803
- R12: footprint C64_PD_PSU:R_0402_1005Metric -> C64_PD_PSU:R_0603_1608Metric; LCSC C25905 -> C23186
- R4, R9: footprint C64_PD_PSU:R_0402_1005Metric -> C64_PD_PSU:R_0603_1608Metric; LCSC C25790 -> C23178
- R6: value 100k -> 75k; footprint C64_PD_PSU:R_0402_1005Metric -> C64_PD_PSU:R_0603_1608Metric; LCSC C25741 -> C23242
- R7: value 13.3k -> 10k; footprint C64_PD_PSU:R_0402_1005Metric -> C64_PD_PSU:R_0603_1608Metric; LCSC C122547 -> C25804
- R8: footprint C64_PD_PSU:R_0402_1005Metric -> C64_PD_PSU:R_0603_1608Metric; LCSC C11702 -> C21190
Other:
- note added: "C64 USB-C PD Power Adapter v0.3 (DC only, no 50/60 Hz: the C64 TOD clock will not tick from mains) Needs a USB-C PD charger offering 15 V (>= 3 A / 45 W recommended). U1 (CH224A) requests 15 V via R1 = 56k. Q1 connects the 15 V rail only after the PD contract (PG low). U2 and U3 start only above ~13.2 V (EN UVLO), so a plain 5 V charger, or one that falls back to 9/12 V, never powers the C64. DIN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"
- note removed: "C64 USB-C PD Power Adapter v0.2 (DC only, no 50/60 Hz: the C64 TOD clock will not tick from mains) Needs a USB-C PD charger offering 15 V (>= 3 A / 45 W recommended). U1 (CH224A) requests 15 V via R1 = 56k. Q1 connects the 15 V rail only after the PD contract (PG low). U2 and U3 start only above ~13.2 V (EN UVLO), so a plain 5 V charger, or one that falls back to 9/12 V, never powers the C64. DIN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"
Changed lines of the file:
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@@
 		(title "C64 USB-C PD Power Adapter")
 		(date "2026-10-27")
-		(rev "0.2")
+		(rev "0.3")
 		(comment 1 "USB-C PD 15 V -> C64 7-pin DIN: +5 V and +12 V DC (on the 9 VAC input), two TPS54302 bucks")
 	)
@@
 			)
 		)
-		(property "Footprint" "C64_PD_PSU:R_0402_1005Metric"
+		(property "Footprint" "C64_PD_PSU:R_0603_1608Metric"
 			(at 124.46 127 0)
 			(effects
@@
 			)
 		)
-		(property "LCSC" "C25796"
+		(property "LCSC" "C23206"
 			(at 124.46 127 0)
 			(effects
@@
 			)
 		)
-		(property "Footprint" "C64_PD_PSU:R_0402_1005Metric"
+		(property "Footprint" "C64_PD_PSU:R_0603_1608Metric"
 			(at 152.4 35.56 0)
 			(effects
@@
 			)
 		)
-		(property "LCSC" "C25741"
+		(property "LCSC" "C25803"
 			(at 152.4 35.56 0)
 			(effects
@@
 			)
 		)
-		(property "Footprint" "C64_PD_PSU:R_0402_1005Metric"
+		(property "Footprint" "C64_PD_PSU:R_0603_1608Metric"
 			(at 152.4 66.04 0)
 			(effects
@@
 			)
 		)
-		(property "LCSC" "C25741"
+		(property "LCSC" "C25803"
 			(at 152.4 66.04 0)
 			(effects
@@
 			)
 		)
-		(property "Footprint" "C64_PD_PSU:R_0402_1005Metric"
+		(property "Footprint" "C64_PD_PSU:R_0603_1608Metric"
 			(at 167.64 127 0)
 			(effects
@@
 			)
 		)
-		(property "LCSC" "C25790"
+		(property "LCSC" "C23178"
 			(at 167.64 127 0)
 			(effects
@@
 			)
 		)
-		(property "Footprint" "C64_PD_PSU:R_0402_1005Metric"
+		(property "Footprint" "C64_PD_PSU:R_0603_1608Metric"
 			(at 167.64 149.86 0)
 			(effects
@@
 			)
 		)
-		(property "LCSC" "C25792"
+		(property "LCSC" "C25819"
 			(at 167.64 149.86 0)
 			(effects
@@
 			)
 		)
-		(property "Value" "100nF"
+		(property "Value" "100nF/50V"
 			(at 228.6 92.71 0)
 			(effects
@@
 			)
 		)
-		(property "Footprint" "C64_PD_PSU:C_0402_1005Metric"
+		(property "Footprint" "C64_PD_PSU:C_0603_1608Metric"
 			(at 226.06 91.44 0)
 			(effects
@@
 			)
 		)
-		(property "LCSC" "C1525"
+		(property "LCSC" "C14663"
 			(at 226.06 91.44 0)
 			(effects
@@
 			)
 		)
-		(property "Footprint" "C64_PD_PSU:L_Changjiang_FXL0630"
+		(property "Footprint" "C64_PD_PSU:L_Changjiang_FXL0530"
 			(at 226.06 111.76 0)
 			(effects
@@
 			)
 		)
-		(property "Description" "cjiang FXL0630-100-M 10 uH 4.5 A / Isat 5.5 A molded, 7x6.6 mm"
+		(property "Description" "cjiang FXL0530-100-M 10 uH 3.2 A / Isat 3.5 A molded, 5.4x5.2 mm (same part as L2: one extended line)"
 			(at 226.06 111.76 0)
 			(effects
@@
 			)
 		)
-		(property "LCSC" "C167223"
+		(property "LCSC" "C177248"
 			(at 226.06 111.76 0)
 			(effects
@@
 			)
 		)
-		(property "Value" "100k"
+		(property "Value" "75k"
 			(at 228.6 138.43 0)
 			(effects
@@
 			)
 		)
-		(property "Footprint" "C64_PD_PSU:R_0402_1005Metric"
+		(property "Footprint" "C64_PD_PSU:R_0603_1608Metric"
 			(at 226.06 137.16 0)
 			(effects
@@
 			)
 		)
-		(property "Description" "FB top: Vout = 0.596 x (1 + 100k/13.3k) = 5.08 V"
+		(property "Description" "FB top: Vout = 0.596 x (1 + 75k/10k) = 5.07 V (Basic values)"
 			(at 226.06 137.16 0)
 			(effects
@@
 			)
 		)
-		(property "LCSC" "C25741"
+		(property "LCSC" "C23242"
 			(at 226.06 137.16 0)
 			(effects
@@
 			)
 		)
-		(property "Value" "13.3k"
+		(property "Value" "10k"
 			(at 228.6 158.75 0)
 			(effects
@@
 			)
 		)
-		(property "Footprint" "C64_PD_PSU:R_0402_1005Metric"
+		(property "Footprint" "C64_PD_PSU:R_0603_1608Metric"
 			(at 226.06 157.48 0)
 			(effects
@@
 			)
 		)
-		(property "LCSC" "C122547"
+		(property "LCSC" "C25804"
 			(at 226.06 157.48 0)
 			(effects
@@
 			)
 		)
-		(property "Value" "75pF"
+		(property "Value" "100pF"
 			(at 213.36 138.43 0)
 			(effects
@@
 			)
 		)
-		(property "Footprint" "C64_PD_PSU:C_0402_1005Metric"
+		(property "Footprint" "C64_PD_PSU:C_0603_1608Metric"
 			(at 210.82 137.16 0)
 			(effects
@@
 			)
 		)
-		(property "LCSC" "C37809"
+		(property "LCSC" "C14858"
 			(at 210.82 137.16 0)
 			(effects
@@
 			)
 		)
-		(property "Footprint" "C64_PD_PSU:R_0402_1005Metric"
+		(property "Footprint" "C64_PD_PSU:R_0603_1608Metric"
 			(at 182.88 254 0)
 			(effects
@@
 			)
 		)
-		(property "LCSC" "C25790"
+		(property "LCSC" "C23178"
 			(at 182.88 254 0)
 			(effects
@@
 			)
 		)
-		(property "Footprint" "C64_PD_PSU:R_0402_1005Metric"
+		(property "Footprint" "C64_PD_PSU:R_0603_1608Metric"
 			(at 182.88 269.24 0)
 			(effects
@@
 			)
 		)
-		(property "LCSC" "C25792"
+		(property "LCSC" "C25819"
 			(at 182.88 269.24 0)
 			(effects
@@
 			)
 		)
-		(property "Value" "100nF"
+		(property "Value" "100nF/50V"
 			(at 228.6 227.33 0)
 			(effects
@@
 			)
 		)
-		(property "Footprint" "C64_PD_PSU:C_0402_1005Metric"
+		(property "Footprint" "C64_PD_PSU:C_0603_1608Metric"
 			(at 226.06 226.06 0)
 			(effects
@@
 			)
 		)
-		(property "LCSC" "C1525"
+		(property "LCSC" "C14663"
 			(at 226.06 226.06 0)
 			(effects
@@
 			)
 		)
-		(property "Footprint" "C64_PD_PSU:R_0402_1005Metric"
+		(property "Footprint" "C64_PD_PSU:R_0603_1608Metric"
 			(at 226.06 256.54 0)
 			(effects
@@
 			)
 		)
-		(property "LCSC" "C25741"
+		(property "LCSC" "C25803"
 			(at 226.06 256.54 0)
 			(effects
@@
 			)
 		)
-		(property "Footprint" "C64_PD_PSU:R_0402_1005Metric"
+		(property "Footprint" "C64_PD_PSU:R_0603_1608Metric"
 			(at 226.06 271.78 0)
 			(effects
@@
 			)
 		)
-		(property "LCSC" "C25905"
+		(property "LCSC" "C23186"
 			(at 226.06 271.78 0)
 			(effects
@@
 			)
 		)
-		(property "Value" "75pF"
+		(property "Value" "100pF"
 			(at 213.36 257.81 0)
 			(effects
@@
 			)
 		)
-		(property "Footprint" "C64_PD_PSU:C_0402_1005Metric"
+		(property "Footprint" "C64_PD_PSU:C_0603_1608Metric"
 			(at 210.82 256.54 0)
 			(effects
@@
 			)
 		)
-		(property "LCSC" "C37809"
+		(property "LCSC" "C14858"
 			(at 210.82 256.54 0)
 			(effects
@@
 	)
 	(symbol
-		(lib_id "C64_PD_PSU:Polyfuse")
+		(lib_id "C64_PD_PSU:R")
 		(at 60.96 162.56 0)
 		(unit 1)
@@
 			)
 		)
-		(property "Value" "2A"
+		(property "Value" "0R"
 			(at 63.5 163.83 0)
 			(effects
@@
 			)
 		)
-		(property "Footprint" "C64_PD_PSU:Fuse_1206_3216Metric"
+		(property "Footprint" "C64_PD_PSU:R_1206_3216Metric"
 			(at 60.96 162.56 0)
 			(effects
@@
 			)
 		)
-		(property "Description" "LUTE 1206L200/16NR PTC, 2 A hold / 3.5 A trip, 16 V"
+		(property "Description" "0 R link (JLC Basic). Optional: fit a 1206 PTC here instead, e.g. LUTE 1206L200/16NR C22374899 (2 A hold)"
 			(at 60.96 162.56 0)
 			(effects
@@
 			)
 		)
-		(property "LCSC" "C22374899"
+		(property "LCSC" "C17888"
 			(at 60.96 162.56 0)
 			(effects
@@
 			)
 		)
-		(property "Description" "TVS 5 V standoff: clamps +5 V and trips F1 if the buck ever fails high"
+		(property "Description" "SMF5.0A TVS (JLC Preferred), clamps +5 V if the buck ever fails high"
 			(at 81.28 175.26 0)
 			(effects
@@
 			)
 		)
-		(property "LCSC" "C193402"
+		(property "LCSC" "C19077497"
 			(at 81.28 175.26 0)
 			(effects
@@
 	)
 	(symbol
-		(lib_id "C64_PD_PSU:Polyfuse")
+		(lib_id "C64_PD_PSU:R")
 		(at 111.76 162.56 0)
 		(unit 1)
@@
 			)
 		)
-		(property "Value" "1.1A"
+		(property "Value" "0R"
 			(at 114.3 163.83 0)
 			(effects
@@
 			)
 		)
-		(property "Footprint" "C64_PD_PSU:Fuse_1206_3216Metric"
+		(property "Footprint" "C64_PD_PSU:R_1206_3216Metric"
 			(at 111.76 162.56 0)
 			(effects
@@
 			)
 		)
-		(property "Description" "BHFUSE BSMD1206-110-24V PTC, 1.1 A hold / 2.2 A trip, 24 V"
+		(property "Description" "0 R link (JLC Basic). Optional: fit a 1206 PTC here instead, e.g. BSMD1206-110-24V C2798026 (1.1 A hold)"
 			(at 111.76 162.56 0)
 			(effects
@@
 			)
 		)
-		(property "LCSC" "C2798026"
+		(property "LCSC" "C17888"
 			(at 111.76 162.56 0)
 			(effects
@@
 			)
 		)
-		(property "Description" "TVS 13 V standoff on the 12 V output"
+		(property "Description" "SMF13A TVS (JLC Preferred) on the 12 V output"
 			(at 132.08 175.26 0)
 			(effects
@@
 			)
 		)
-		(property "LCSC" "C353315"
+		(property "LCSC" "C41376087"
 			(at 132.08 175.26 0)
 			(effects
@@
 			)
 		)
-		(property "Footprint" "C64_PD_PSU:R_0402_1005Metric"
+		(property "Footprint" "C64_PD_PSU:R_0603_1608Metric"
 			(at 101.6 187.96 0)
 			(effects
@@
 			)
 		)
-		(property "LCSC" "C11702"
+		(property "LCSC" "C21190"
 			(at 101.6 187.96 0)
 			(effects
@@
 		)
 	)
-	(text "C64 USB-C PD Power Adapter v0.2 (DC only, no 50/60 Hz: the C64 TOD clock will not tick from mains)\nNeeds a USB-C PD charger offering 15 V (>= 3 A / 45 W recommended). U1 (CH224A) requests 15 V via R1 = 56k.\nQ1 connects the 15 V rail only after the PD contract (PG low). U2 and U3 start only above ~13.2 V (EN UVLO),\nso a plain 5 V charger, or one that falls back to 9/12 V, never powers the C64.\nDIN: 4+5 = +5.08 V (U2, F1 2 A PTC, D1 TVS), 6 = +12.3 V DC (U3, F2 1.1 A PTC, D2 TVS) into the C64 \"9 VAC\" bridge, 1/2/3/7 = GND.\n12 V DC = the peak of the stock 9 VAC, so user port pins 10/11 see no more than an original PSU gives (but DC, not AC)."
+	(text "C64 USB-C PD Power Adapter v0.3 (DC only, no 50/60 Hz: the C64 TOD clock will not tick from mains)\nNeeds a USB-C PD charger offering 15 V (>= 3 A / 45 W recommended). U1 (CH224A) requests 15 V via R1 = 56k.\nQ1 connects the 15 V rail only after the PD contract (PG low). U2 and U3 start only above ~13.2 V (EN UVLO),\nso a plain 5 V charger, or one that falls back to 9/12 V, never powers the C64.\nDIN: 4+5 = +5.08 V (U2, D1 TVS), 6 = +12.3 V DC (U3, D2 TVS) into the C64 \"9 VAC\" bridge, 1/2/3/7 = GND.\n12 V DC = the peak of the stock 9 VAC, so user port pins 10/11 see no more than an original PSU gives (but DC, not AC)."
 		(exclude_from_sim no)
 		(at 25.4 22.86 0)
